File: pcb_fingerboard/neopixel1515.kicad_pcb (KiCad board)
At the start: 2 copper layers, 330 x 45 mm, 122 parts

Commit message: Layout fingerboard dimension
Parts:
- added J1: Conn_01x03, Connector_PinHeader_2.54mm:PinHeader_1x03_P2.54mm_Horizontal, F.Cu at (326.0, 21.0)
- moved C1 307.5 mm to (316.3, 26.0), turned to 90 degrees
- moved R1 274.2 mm to (291.0, 43.0)
- moved D120 266.0 mm to (287.0, 43.0), turned to 180 degrees
- moved D60 265.0 mm to (287.0, 23.0), turned to 180 degrees
- moved D119 259.3 mm to (283.3, 43.0), turned to 180 degrees
- moved D59 258.4 mm to (283.3, 23.0), turned to 180 degrees
- moved D118 252.5 mm to (279.4, 43.0), turned to 180 degrees
- moved D58 251.5 mm to (279.4, 23.0), turned to 180 degrees
- moved D117 245.4 mm to (275.3, 43.0), turned to 180 degrees
- moved D57 244.4 mm to (275.3, 23.0), turned to 180 degrees
- moved D116 238.1 mm to (271.0, 43.0), turned to 180 degrees
- moved D56 237.0 mm to (271.0, 23.0), turned to 180 degrees
- moved D115 230.5 mm to (266.4, 43.0), turned to 180 degrees
- moved D55 229.4 mm to (266.4, 23.0), turned to 180 degrees
- moved D114 222.7 mm to (261.5, 43.0), turned to 180 degrees
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- renumbered D91 to D1, D100 to D10, D21 to D100, D20 to D101, D19 to D102, D18 to D103, D17 to D104, D16 to D105, D15 to D106, D14 to D107, D13 to D108, D12 to D109, D101 to D11, D11 to D110, D10 to D111, D9 to D112, D8 to D113, D7 to D114, D6 to D115, D5 to D116, D4 to D117, D3 to D118, D2 to D119, D102 to D12, D1 to D120, D103 to D13, D104 to D14, D105 to D15, D106 to D16, D107 to D17, D108 to D18, D109 to D19, D92 to D2, D110 to D20, D111 to D21, D112 to D22, D113 to D23, D114 to D24, D115 to D25, D116 to D26, D117 to D27, D118 to D28, D119 to D29, D93 to D3, D120 to D30, D90 to D31, D89 to D32, D88 to D33, D87 to D34, D86 to D35, D85 to D36, D84 to D37, D83 to D38, D82 to D39, D94 to D4, D81 to D40, D80 to D41, D79 to D42, D78 to D43, D77 to D44, D76 to D45, D75 to D46, D74 to D47, D73 to D48, D72 to D49, D95 to D5, D71 to D50, D70 to D51, D69 to D52, D68 to D53, D67 to D54, D66 to D55, D65 to D56, D64 to D57, D63 to D58, D62 to D59, D96 to D6, D61 to D60, D31 to D61, D32 to D62, D33 to D63, D34 to D64, D35 to D65, D36 to D66, D37 to D67, D38 to D68, D39 to D69, D97 to D7, D40 to D70, D41 to D71, D42 to D72, D43 to D73, D44 to D74, D45 to D75, D46 to D76, D47 to D77, D48 to D78, D49 to D79, D98 to D8, D50 to D80, D51 to D81, D52 to D82, D53 to D83, D54 to D84, D55 to D85, D56 to D86, D57 to D87, D58 to D88, D59 to D89, D99 to D9, D60 to D90, D30 to D91, D29 to D92, D28 to D93, D27 to D94, D26 to D95, D25 to D96, D24 to D97, D23 to D98, D22 to D99
Connections:
- D1 pad 1: Net-(D91-Pad1) (its old number) -> Net-(D1-Pad1)
- D120 pad 1: Net-(D1-Pad1) -> Net-(D120-Pad1)
- D30 pad 3: Net-(D120-Pad3) -> Net-(D30-Pad3)
- D31 pad 3: Net-(D31-Pad1) (its old number) -> Net-(D1-Pad1)
- D60 pad 1: Net-(D120-Pad3) -> Net-(D60-Pad1)
- D61 pad 1: Net-(D31-Pad1) (its old number) -> Net-(D61-Pad1)
- D90 pad 3: Net-(D1-Pad1) -> Net-(D60-Pad1)
- D91 pad 3: Net-(D30-Pad3) -> Net-(D61-Pad1)
- R1 pad 1: Net-(R1-Pad1) -> Net-(D120-Pad1)
- R1 pad 2: Net-(D91-Pad1) (its old number) -> Net-(J1-Pad2)
Routing:
- net GND: track 0.00 -> 169.7 mm, vias 0 -> 120
- net Net-(J1-Pad2): track 0.00 -> 46.4 mm
- net Net-(D91-Pad1): track 0.00 -> 17.9 mm
- net Net-(D61-Pad3): track 0.00 -> 17.9 mm
- net Net-(D31-Pad1): track 0.00 -> 17.9 mm
- net Net-(D1-Pad3): track 0.00 -> 17.9 mm
- net Net-(D62-Pad3): track 0.00 -> 16.9 mm
- net Net-(D92-Pad1): track 0.00 -> 16.9 mm
- net Net-(D32-Pad1): track 0.00 -> 16.9 mm
- net Net-(D2-Pad3): track 0.00 -> 16.9 mm
- net Net-(D93-Pad1): track 0.00 -> 15.9 mm
- net Net-(D63-Pad3): track 0.00 -> 15.9 mm
- net Net-(D33-Pad1): track 0.00 -> 15.9 mm
- net Net-(D3-Pad3): track 0.00 -> 15.9 mm
- net Net-(D94-Pad1): track 0.00 -> 15.0 mm
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- added copper zone on B.Cu, net GND
- added copper zone on F.Cu, net VDD
Other:
- board size 330 x 45 mm -> 330 x 43 mm

Commit message: Pre-print fingerboard pcb
Parts:
- added G***: LOGO, victor:logo_mini, F.Cu at (334.0, 7.00)
- added H1: MountingHole, MountingHole:MountingHole_3.2mm_M3, F.Cu at (4.00, 7.00)
- added H2: MountingHole, MountingHole:MountingHole_3.2mm_M3, F.Cu at (341.0, 7.00)
- added H3: MountingHole, MountingHole:MountingHole_3.2mm_M3, F.Cu at (4.00, 41.0)
- added H4: MountingHole, MountingHole:MountingHole_3.2mm_M3, F.Cu at (341.0, 41.0)
- moved C1 15.0 mm to (331.3, 26.5)
- moved J1 15.0 mm to (341.0, 21.5)
Routing:
- net Net-(J1-Pad2): track 46.4 -> 59.3 mm
Other:
- board size 330 x 43 mm -> 345 x 42 mm
- board text added: "v1.0"

Commit message: Added padded mounting holes with vias
Parts:
- H1, H2, H3, H4: value MountingHole -> MountingHole_Pad; footprint MountingHole:MountingHole_3.2mm_M3 -> MountingHole:MountingHole_3.2mm_M3_Pad_Via
- moved G*** 2.00 mm to (332.0, 7.00)
- moved H1 1.41 mm to (5.00, 8.00), turned to 180 degrees
- moved H2 1.41 mm to (340.0, 8.00), turned to 180 degrees
- moved H3 1.41 mm to (5.00, 40.0)
- moved H4 1.41 mm to (340.0, 40.0)
Connections:
- H1 pad 1: (no net) -> GND
- H2 pad 1: (no net) -> GND
- H3 pad 1: (no net) -> GND
- H4 pad 1: (no net) -> GND
